Commit message: update robot1_description

File: robot1_description/urdf/robot1.urdf (robot description, URDF)
Before this commit: robot origins, 12 links, 11 joints
Links:
- link left_gripper: geometry collision box size=0.1 .1 .1; visual mesh filename=package://robot1_description/meshes/gripper_v0/l_finger.dae
- link left_tip: geometry collision box size=0.1 .1 .1; visual mesh filename=package://robot1_description/meshes/gripper_v0/l_finger_tip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
- link right_gripper: geometry collision box size=0.1 .1 .1; visual mesh filename=package://robot1_description/meshes/gripper_v0/l_finger.dae
- link right_tip: geometry collision box size=0.1 .1 .1; visual mesh filename=package://robot1_description/meshes/gripper_v0/l_finger_tip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

File: robot1_description/urdf/robot1.xacro (robot description, xacro)
@@ -207,5 +207,5 @@
       <origin rpy="0 0 0" xyz="0 0 0"/>
       <geometry>
-        <mesh filename="package://pr2_description/meshes/gripper_v0/l_finger.dae"/>
+        <mesh filename="package://robot1_description/meshes/gripper_v0/l_finger.dae"/>
       </geometry>
     </visual>
@@ -225,5 +225,5 @@
       <origin rpy="0.0 0 0" xyz="0.09137 0.00495 0"/>
       <geometry>
-        <mesh filename="package://pr2_description/meshes/gripper_v0/l_finger_tip.dae"/>
+        <mesh filename="package://robot1_description/meshes/gripper_v0/l_finger_tip.dae"/>
       </geometry>
     </visual>
@@ -246,5 +246,5 @@
       <origin rpy="-3.1415 0 0" xyz="0 0 0"/>
       <geometry>
-        <mesh filename="package://pr2_description/meshes/gripper_v0/l_finger.dae"/>
+        <mesh filename="package://robot1_description/meshes/gripper_v0/l_finger.dae"/>
       </geometry>
     </visual>
@@ -264,5 +264,5 @@
       <origin rpy="-3.1415 0 0" xyz="0.09137 0.00495 0"/>
       <geometry>
-        <mesh filename="package://pr2_description/meshes/gripper_v0/l_finger_tip.dae"/>
+        <mesh filename="package://robot1_description/meshes/gripper_v0/l_finger_tip.dae"/>
       </geometry>
     </visual>

File: robot1_description/urdf/robot1_arm.xacro (robot description, xacro)
@@ -86,5 +86,5 @@
       <origin rpy="0 0 0" xyz="0 0 0"/>
       <geometry>
-        <mesh filename="package://pr2_description/meshes/gripper_v0/l_finger.dae"/>
+        <mesh filename="package://robot1_description/meshes/gripper_v0/l_finger.dae"/>
       </geometry>
     </visual>
@@ -104,5 +104,5 @@
       <origin rpy="0.0 0 0" xyz="0.09137 0.00495 0"/>
       <geometry>
-        <mesh filename="package://pr2_description/meshes/gripper_v0/l_finger_tip.dae"/>
+        <mesh filename="package://robot1_description/meshes/gripper_v0/l_finger_tip.dae"/>
       </geometry>
     </visual>
@@ -125,5 +125,5 @@
       <origin rpy="-3.1415 0 0" xyz="0 0 0"/>
       <geometry>
-        <mesh filename="package://pr2_description/meshes/gripper_v0/l_finger.dae"/>
+        <mesh filename="package://robot1_description/meshes/gripper_v0/l_finger.dae"/>
       </geometry>
     </visual>
@@ -143,5 +143,5 @@
       <origin rpy="-3.1415 0 0" xyz="0.09137 0.00495 0"/>
       <geometry>
-        <mesh filename="package://pr2_description/meshes/gripper_v0/l_finger_tip.dae"/>
+        <mesh filename="package://robot1_description/meshes/gripper_v0/l_finger_tip.dae"/>
       </geometry>
     </visual>

File: robot1_description/urdf/robot1_physics.urdf (robot description, URDF)
Before this commit: robot origins, 12 links, 11 joints
Links:
- link left_gripper: geometry collision box size=0.1 .1 .1; visual mesh filename=package://robot1_description/meshes/gripper_v0/l_finger.dae
- link left_tip: geometry collision box size=0.1 .1 .1; visual mesh filename=package://robot1_description/meshes/gripper_v0/l_finger_tip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
- link right_gripper: geometry collision box size=0.1 .1 .1; visual mesh filename=package://robot1_description/meshes/gripper_v0/l_finger.dae
- link right_tip: geometry collision box size=0.1 .1 .1; visual mesh filename=package://robot1_description/meshes/gripper_v0/l_finger_tip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
